File: _autosave-Amini_Kicad_Lock.kicad_sch (KiCad schematic)
At the start: 40 parts, among them J1 Conn_01x02_Pin, J2 Conn_01x04, J3 MM8130-2600RA2, J4 Conn_01x03_Pin, U1 nRF5340-QKxx, X1 ${ALTIUM_VALUE}, X2 ${ALTIUM_VALUE}

Commit message: backup mid routing
Parts:
- L2: footprint INDC1608X06L -> Inductor_SMD:L_0603_1608Metric
Changed lines of the file:
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@@
 			)
 		)
-		(property "Footprint" "INDC1608X06L"
+		(property "Footprint" "Inductor_SMD:L_0603_1608Metric"
 			(at 50.8 85.09 0)
 			(effects
