File: Amini_Lock.kicad_sch (KiCad schematic)
At the start: 42 parts, among them J1 Conn_01x02_Pin, J2 Conn_01x04, J3 Conn_01x04_Pin, U1 nRF5340-QKxx, X1 ${ALTIUM_VALUE}, X2 ${ALTIUM_VALUE}

Commit message: Adding V1.1
Parts:
- removed C17: 0.7pF, Capacitor_SMD:C_0402_1005Metric_Pad0.74x0.62mm_HandSolder, symbol Device:C
- removed D1: D, Diode_SMD:D_0402_1005Metric_Pad0.77x0.64mm_HandSolder, symbol Device:D
- removed J1: Conn_01x02_Pin, Connector_PinHeader_2.00mm:PinHeader_1x02_P2.00mm_Vertical, symbol Connector:Conn_01x02_Pin
- removed J3: Conn_01x04_Pin, Connector_PinHeader_2.00mm:PinHeader_1x04_P2.00mm_Vertical, symbol Connector:Conn_01x04_Pin
- removed L4: 2.2nH, Capacitor_SMD:C_0402_1005Metric_Pad0.74x0.62mm_HandSolder, symbol Device:L
- removed TPclk1, TPgnd1, TPio1, TPset1: TestPoint, TestPoint:TestPoint_Pad_D1.5mm, symbol Connector:TestPoint
- added C17: ${ALTIUM_VALUE}, CAPC0603X03L_C, symbol nrf5340_qkaa_config3-altium-import:root_3_CAP
- added C20: ${ALTIUM_VALUE}, CAPC0603X03L_C, symbol pca10143_sheet2_nrf5340_mcu-altium-import:root_1_CAP
- added J1: Conn_01x02, Connector_JST:JST_SH_BM02B-SRSS-TB_1x02-1MP_P1.00mm_Vertical, symbol Connector_Generic:Conn_01x02
- added L4: ${ALTIUM_VALUE}, INDC0603X03L_C, symbol pca10143_sheet2_nrf5340_mcu-altium-import:root_0_mirrored_IND
- added TP1, TP2: TestPoint_Alt, TestPoint:TestPoint_Pad_1.5x1.5mm, symbol Connector:TestPoint_Alt
- added TP10, TP11, TP13, TP16, TP18, TP6, TP7, TP8, TP9: TestPoint_Alt, TestPoint:TestPoint_THTPad_2.0x2.0mm_Drill1.0mm, symbol Connector:TestPoint_Alt
- added TP12: TestPoint, TestPoint:TestPoint_Pad_1.0x1.0mm, symbol Connector:TestPoint
- added TP3, TP4, TP5: TestPoint, TestPoint:TestPoint_Pad_D1.0mm, symbol Connector:TestPoint
- added U2: ${ALTIUM_VALUE}, SON127P600X80_HS-9N, symbol 400432-altium-import:root_0_MX25R6435FZNIL0
- C1: value N.C -> ${ALTIUM_VALUE}; footprint Capacitor_SMD:C_0402_1005Metric_Pad0.74x0.62mm_HandSolder -> CAPC0603X03L_C
- C18: footprint Capacitor_SMD:C_0402_1005Metric_Pad0.74x0.62mm_HandSolder -> CAPC0603X03L_C_NC
- C19: footprint Capacitor_SMD:C_0402_1005Metric_Pad0.74x0.62mm_HandSolder -> Capacitor_SMD:C_0201_0603Metric_Pad0.64x0.40mm_HandSolder
- C7: footprint Capacitor_SMD:C_0402_1005Metric -> CAPC1005X04L
- J2: footprint Connector_PinHeader_2.54mm:PinHeader_2x02_P2.54mm_Vertical -> Connector_JST:JST_SH_SM04B-SRSS-TB_1x04-1MP_P1.00mm_Horizontal
- L1: value 0R -> ${ALTIUM_VALUE}; footprint Capacitor_SMD:C_0402_1005Metric_Pad0.74x0.62mm_HandSolder -> INDC0603X03L_C; ALTIUM_VALUE (none) -> 2.2nH; AUTHOR (none) -> rsk; COMPONENT CLASS (none) -> Inductors; COMPONENT STATUS (none) -> Active; COMPONENTLINK1DESCRIPTION (none) -> Datasheet; COMPONENTLINK1URL (none) -> https://search.murata.co.jp/Ceramy/image/img/P02/JELF243C-0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; COMPONENTLINK2DESCRIPTION (none) -> Supplier link; FOOTPRINT DOC (none) -> 0201; HELPURL (none) -> https://psearch.en.murata.com/inductor/product/LQP03HQ2N2B0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; LATESTREVISIONDATE (none) -> 2018-10-23; MANUFACTURER (none) -> Murata; MANUFACTURER PART NUMBER 0 -> LQP03HQ2N2B02; NOTE (none) -> -55°C ~ 125°C; PAD COUNT (none) -> 2; PART NUMBER 0 -> L0201-2n2-HQ-Murata; PART NUMBER NEMS (none) -> 100300209; PART NUMBER NORAUTRON (none) -> 26521773; PARTID (none) -> 100300209; PUBLISHED (none) -> 2018-10-23; SUPPLIER 1 (none) -> Digi-Key; SUPPLIER 2 (none) -> N.A.; SUPPLIER PART NUMBER 1 (none) -> 490-13899-1-ND
- L2: footprint Nordic_Semiconductor:INDC1608X06L -> INDC1608X06L
Connections:
- net GND: now also C17.2, C20.1, J1.1 (Pin_1), TP1.1, TP16.1, U2.4 (GND)
- net SWDCLK: now also TP3.1
- net SWDIO: now also TP4.1
- net VDD_nRF: now also C17.1, J1.2 (Pin_2), TP18.1, TP2.1, U2.8 (VCC)
- net ~{RESET}: now also TP5.1
- net at C1.2, L1.1: now also U1.L31 (ANT); no longer C19.2
- net at C18.2, L1.2: now also C19.2, L4.2, TP12.1; no longer A1.1
- net P0.28/AIN7: now reaches U1.AE31 (AIN7/P0.28)
- net P0.28/AIN7: now also LED1.1 (C), TP9.1
- net at U1.AK10 (IO2/P0.15): now also U2.3 (SIO2/~{WP})
- net at U1.AK12 (SCK/P0.17): now also U2.6 (SCLK)
- net at U1.AK14 (CSN/P0.18): now also U2.1 (~{CS})
- net at U1.AK30 (AIN6/P0.27): now also TP10.1
- net at U1.AK8 (IO1/P0.14): now also U2.2 (SIO1/SO)
- net at U1.AL5 (IO0/P0.13): now also U2.5 (SIO0/SI)
- net at U1.AL9 (IO3/P0.16): now also U2.7 (SIO3/~{RESET})
- net at U1.B22 (P0.31): now also TP6.1
- net P0.30: now reaches U1.B24 (P0.30)
- net P0.30: now also LED3.1 (C), TP7.1
- net P0.29: now reaches U1.U31 (P0.29)
- net P0.29: now also LED2.1 (C), TP8.1
- net LED1: no longer names the net of U1.W1 (NFC1/P0.02)
- net LED1: no longer LED3.1 (C)
- net LED2: no longer names the net of U1.AL27 (P0.24)
- net LED2: now also TP13.1; no longer LED2.1 (C)
- net LED3: no longer names the net of U1.AL29 (AIN5/P0.26)
- net LED3: now also TP11.1; no longer LED1.1 (C)
- net MIC: no longer names the net of U1.AA1 (NFC2/P0.03)
- new net: A1.1, C20.2, L4.1
Other:
- note added: "Amini Lock v1"
- note removed: "Amini Lock V2"
- note removed: "Diagnostic Leds"
- note removed: "Power Interface"
- note removed: "Programing interface"
- title: Amini Lock -> (none)
